Commit message: changes to work with sick urdf

File: sick_visionary_t_driver/description/urdf/visionary_t.urdf.xacro (robot description, xacro)
@@ -1,8 +1,8 @@
 <?xml version="1.0"?>
-<robot name="r3_mill_tool" xmlns:xacro="http://wiki.ros.org/xacro">
+<robot xmlns:xacro="http://www.ros.org/wiki/xacro" name="sick_visionary_t">
+  <xacro:include filename="$(find sick_visionary_t_driver)/description/urdf/visionary_t_macro.urdf.xacro" />
   <link name="base_link"/>
-  <xacro:include filename="$(find sick_visionary_t_driver)/description/urdf/visionary_t_macro.urdf.xacro" />
   <xacro:sick_visionary_t parent="base_link" has_holder="true" holder_tilt="${-25/180*pi}">
-    <origin xyz="0.085 0 1.85" rpy="${pi} 0 0" />
+    <origin xyz="0.0 0 0.0" rpy="0 0 0" />
   </xacro:sick_visionary_t>
 </robot>

File: sick_visionary_t_driver/description/urdf/visionary_t_macro.urdf.xacro (robot description, xacro)
@@ -1,3 +1,4 @@
-<robot xmlns:xacro="http://wiki.ros.org/xacro">
+<?xml version="1.0"?>
+<robot xmlns:xacro="http://www.ros.org/wiki/xacro">
     <xacro:macro name="sick_visionary_t" params="parent *origin has_holder holder_tilt">
         <xacro:if value="${has_holder}">
